File: keyboard_layout_jopr_v01.kicad_pcb (KiCad board)
At the start: 2 copper layers, 428.6 x 120.7 mm, 228 parts, among them SW1 SW_Push, U1 ATmega32U4-AU, Y1 16MHz

Commit message: Inter-key tracks and USB Data tracks only
Parts:
- moved USB1 278.6 mm to (397.7, 15.1)
- moved F1 275.0 mm to (392.2, 26.5)
- moved R2 262.1 mm to (398.8, 24.6), turned to 90 degrees
- moved R3 259.4 mm to (396.1, 24.6), turned to 90 degrees
- moved C6 34.9 mm to (401.0, 72.2)
- moved R4 34.9 mm to (406.4, 68.3)
- moved C3 34.9 mm to (387.4, 62.7)
- moved C4 34.9 mm to (406.4, 59.5)
- moved C5 34.9 mm to (390.5, 54.7)
- moved C7 34.9 mm to (387.6, 69.3)
- moved U1 34.9 mm to (396.9, 63.5)
- moved C1 33.6 mm to (401.6, 50.8)
- moved C2 33.6 mm to (392.1, 50.8)
- moved Y1 33.6 mm to (396.9, 50.8)
- moved R1 17.4 mm to (429.4, 42.1)
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- renumbered D_P5 to D_O5, MX_P5 to MX_O5
Connections:
- MX_O5 pad 1: COL_P -> COL_O
Routing:
- net COL_A: track 108.7 -> 555.8 mm, vias 0 -> 2
- net COL_B: track 111.9 -> 538.7 mm, vias 0 -> 2
- net COL_C: track 115.4 -> 517.0 mm, vias 0 -> 2
- net COL_D: track 92.0 -> 476.3 mm, vias 0 -> 2
- net COL_E: track 92.0 -> 454.6 mm, vias 0 -> 2
- net GND: track 8.90 -> 310.4 mm, vias 2 -> 8
- net COL_F: track 93.7 -> 382.7 mm, vias 0 -> 3
- net COL_G: track 111.4 -> 378.5 mm, vias 0 -> 3
- net COL_H: track 94.3 -> 345.4 mm, vias 0 -> 3
- net COL_I: track 96.1 -> 320.7 mm, vias 0 -> 3
- net Net-(R2-Pad1): track 267.5 -> 52.9 mm
- net Net-(R3-Pad1): track 267.9 -> 53.6 mm
- net COL_J: track 122.6 -> 335.4 mm, vias 0 -> 3
- net COL_K: track 126.8 -> 317.9 mm, vias 0 -> 4
- net COL_N: track 84.6 -> 263.6 mm, vias 0 -> 2
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- added copper zone on B.Cu, net GND
Other:
- board size 428.6 x 120.7 mm -> 433.4 x 123.8 mm
