File: keyboard_layout_jopr.kicad_pcb (KiCad board)
At the start: 2 copper layers, 433.4 x 123.8 mm, 228 parts, among them SW1 SW_Push, U1 ATmega32U4-AU, Y1 16MHz

Commit message: Inter-key tracks and USB Data tracks only
Parts:
- moved USB1 278.6 mm to (119.1, 17.6)
- moved F1 275.0 mm to (117.2, 32.6)
- moved R2 262.1 mm to (136.7, 17.2), turned to 180 degrees
- moved R3 259.4 mm to (136.7, 19.6), turned to 180 degrees
- moved C5 35.0 mm to (391.3, 19.8)
- moved C6 34.9 mm to (401.8, 37.3)
- moved R4 34.9 mm to (407.2, 33.3)
- moved C3 34.9 mm to (388.1, 27.8)
- moved C4 34.9 mm to (407.2, 24.6)
- moved C7 34.9 mm to (388.4, 34.4)
- moved U1 34.9 mm to (397.7, 28.6)
- moved C1 33.6 mm to (405.6, 17.5)
- moved C2 33.6 mm to (396.1, 17.5)
- moved Y1 33.6 mm to (400.8, 17.5)
- moved R1 17.4 mm to (422.3, 26.2)
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- renumbered D_O5 to D_P5, MX_O5 to MX_P5
Connections:
- MX_P5 pad 1: COL_O -> COL_P
Routing:
- net COL_A: track 555.8 -> 108.7 mm, vias 2 -> 0
- net COL_B: track 538.7 -> 111.9 mm, vias 2 -> 0
- net COL_C: track 517.0 -> 115.4 mm, vias 2 -> 0
- net COL_D: track 476.3 -> 92.0 mm, vias 2 -> 0
- net COL_E: track 454.6 -> 92.0 mm, vias 2 -> 0
- net GND: track 304.9 -> 8.90 mm, vias 6 -> 2
- net COL_F: track 382.7 -> 93.7 mm, vias 3 -> 0
- net COL_G: track 378.5 -> 111.4 mm, vias 3 -> 0
- net COL_H: track 345.4 -> 94.3 mm, vias 3 -> 0
- net COL_I: track 320.7 -> 96.1 mm, vias 3 -> 0
- net Net-(R2-Pad1): track 52.9 -> 267.5 mm
- net Net-(R3-Pad1): track 53.6 -> 267.9 mm
- net COL_J: track 335.4 -> 122.6 mm, vias 3 -> 0
- net COL_K: track 317.9 -> 126.8 mm, vias 4 -> 0
- net COL_N: track 263.6 -> 84.6 mm, vias 2 -> 0
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Other:
- board size 433.4 x 123.8 mm -> 428.6 x 120.7 mm

Commit message: maybe better tracks
Parts:
- moved SW1 30.5 mm to (398.9, 26.8), turned to 90 degrees
- moved U1 23.0 mm to (410.2, 47.9)
- moved C7 23.0 mm to (401.0, 53.7)
- moved C3 23.0 mm to (400.7, 47.1)
- moved C6 23.0 mm to (414.4, 56.6)
- moved R4 23.0 mm to (419.8, 52.6)
- moved C4 23.0 mm to (419.8, 43.9)
- moved C5 23.0 mm to (403.9, 39.1)
- moved C1 22.9 mm to (416.9, 37.4)
- moved C2 22.9 mm to (407.4, 37.4)
- moved Y1 22.9 mm to (412.1, 37.4)
- moved R1 21.9 mm to (401.8, 34.0), turned to 180 degrees
Connections:
- U1 pad 1: COL_K -> Net-(U1-Pad1)
- U1 pad 10: COL_H -> COL_R
- U1 pad 11: COL_G -> COL_Q
- U1 pad 12: COL_F -> COL_R
- U1 pad 18: COL_E -> ROW4
- U1 pad 19: COL_D -> ROW3
- U1 pad 20: COL_C -> ROW1
- U1 pad 21: COL_B -> COL_P
- U1 pad 22: COL_A -> COL_M
- U1 pad 25: ROW0 -> COL_N
- U1 pad 26: COL_S -> COL_O
- U1 pad 27: ROW1 -> COL_K
- U1 pad 28: COL_R -> COL_L
- U1 pad 29: ROW2 -> COL_J
- U1 pad 30: COL_Q -> COL_G
- U1 pad 31: COL_P -> COL_C
- U1 pad 32: ROW3 -> COL_B
- U1 pad 36: ROW5 -> COL_A
- U1 pad 37: COL_O -> COL_I
- U1 pad 38: COL_N -> COL_H
- U1 pad 39: ROW4 -> COL_F
- U1 pad 40: COL_M -> COL_E
- U1 pad 41: COL_L -> COL_D
- U1 pad 8: COL_J -> COL_S
- U1 pad 9: COL_I -> ROW5
Routing:
- net COL_A: track 108.7 -> 541.6 mm, vias 0 -> 4
- net COL_B: track 111.9 -> 543.8 mm, vias 0 -> 4
- net COL_C: track 115.4 -> 526.5 mm, vias 0 -> 4
- net +5V: track 0.00 -> 383.3 mm, vias 0 -> 7
- net COL_D: track 92.0 -> 450.8 mm, vias 0 -> 4
- net COL_G: track 111.4 -> 450.3 mm, vias 0 -> 4
- net COL_E: track 92.0 -> 416.7 mm, vias 0 -> 2
- net COL_F: track 93.7 -> 393.9 mm, vias 0 -> 2
- net COL_J: track 122.6 -> 391.6 mm, vias 0 -> 4
- net COL_H: track 94.3 -> 359.8 mm, vias 0 -> 2
- net COL_K: track 126.8 -> 378.0 mm, vias 0 -> 2
- net COL_I: track 96.1 -> 346.5 mm, vias 0 -> 2
- net COL_N: track 84.6 -> 321.5 mm, vias 0 -> 1
- net COL_M: track 127.1 -> 357.7 mm, vias 0 -> 1
- net COL_L: track 137.7 -> 361.1 mm, vias 2 -> 6
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- added copper zone on B.Cu, net GND
