File: keyboard_layout_jopr.kicad_pcb (KiCad board)
At the start: 2 copper layers, 428.6 x 120.7 mm, 228 parts, among them SW1 SW_Push, U1 ATmega32U4-AU, Y1 16MHz

Commit message: replaced MX_Hybrid with MX_Only footprints
Parts:
- MX_A0, MX_A1, MX_B0, MX_B1, MX_B2, MX_B3, MX_B4, MX_C0, MX_C1, MX_C2, MX_C3, MX_C4, MX_D0, MX_D1, MX_D2, MX_D3, MX_D4, MX_E0, MX_E1, MX_E2, MX_E3, MX_E4, MX_F0, MX_F1, MX_F2, MX_F3, MX_F4, MX_G0, MX_G1, MX_G2, MX_G3, MX_G4, MX_H0, MX_H1, MX_H2, MX_H3, MX_H4, MX_I0, MX_I1, MX_I2, MX_I3, MX_I4, MX_J0, MX_J1, MX_J2, MX_J3, MX_J4, MX_K0, MX_K1, MX_K2, MX_K3, MX_K4, MX_L0, MX_L1, MX_L2, MX_L3, MX_L4, MX_M0, MX_M1, MX_M2, MX_M3, MX_N0, MX_N4, MX_O1, MX_O2, MX_O3, MX_O4, MX_P1, MX_P2, MX_P3, MX_P4, MX_P5, MX_Q1, MX_Q2, MX_Q3, MX_Q5, MX_R0, MX_R1, MX_R3, MX_R4, MX_R5, MX_S0, MX_S1, MX_S3, MX_S4, MX_S5: footprint MX_Alps_Hybrid:MX-1U-NoLED -> MX_Only:MXOnly-1U-NoLED
- MX_A2: footprint MX_Alps_Hybrid:MX-1.5U-NoLED -> MX_Only:MXOnly-1.5U-NoLED
- MX_A3: footprint MX_Alps_Hybrid:MX-1.75U-NoLED -> MX_Only:MXOnly-1.75U-NoLED
- MX_A4, MX_A5, MX_B5, MX_C5, MX_J5, MX_K5, MX_L5, MX_M5: footprint MX_Alps_Hybrid:MX-1.25U-NoLED -> MX_Only:MXOnly-1.25U-NoLED
- MX_G5: footprint MX_Alps_Hybrid:MX-6.25U-NoLED -> MX_Only:MXOnly-6.25U-NoLED
- MX_M4: footprint MX_Alps_Hybrid:MX-2.75U-NoLED -> MX_Only:MXOnly-2.75U-NoLED
- MX_N1, MX_N5, MX_Q4, MX_R2: footprint MX_Alps_Hybrid:MX-2U-NoLED -> MX_Only:MXOnly-2U-NoLED
- MX_N3: footprint MX_Alps_Hybrid:MX-ISO -> MX_Only:MXOnly-ISO-NoLED
- MX_O0, MX_P0, MX_Q0: footprint MX_Alps_Hybrid:MX-1U -> MX_Only:MXOnly-1U
Routing:
- net COL_G: track 450.3 -> 457.7 mm
- net COL_P: track 292.6 -> 299.7 mm
- net COL_J: track 391.6 -> 398.1 mm
- net COL_Q: track 189.1 -> 194.1 mm
- net COL_K: track 378.0 -> 382.0 mm
- net COL_B: track 543.8 -> 547.8 mm
- net COL_F: track 393.9 -> 397.8 mm
- net COL_C: track 526.5 -> 530.4 mm
- net COL_O: track 297.1 -> 300.7 mm
- net COL_S: track 173.8 -> 177.4 mm
- net COL_D: track 450.8 -> 454.3 mm
- net COL_L: track 361.1 -> 364.1 mm
- net COL_H: track 359.8 -> 361.8 mm
- net COL_E: track 416.7 -> 418.7 mm
- net COL_R: track 293.4 -> 295.0 mm
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
Commit message: added ESD-protection
Parts:
- added U2: TPD4EUSB30, SOT65P210X110-6N:SOT65P210X110-6N, B.Cu at (122.2, 28.6)
- MX_O0, MX_P0, MX_Q0: value MX-LED -> MX-NoLED; footprint MX_Only:MXOnly-1U -> MX_Only:MXOnly-1U-NoLED
Routing:
- net GND: track 124.5 -> 406.4 mm, vias 6 -> 8
- net D+: track 25.9 -> 30.2 mm, vias 0 -> 2
- net ROW0: track 481.2 -> 483.4 mm
- net D-: track 27.1 -> 28.3 mm

Commit message: squared matrix, updated and renamed PDFs
Parts:
- U2: value TPD4EUSB30 -> SOT65P210X110
- moved C1 4.25 mm to (416.9, 33.1)
- moved Y1 4.13 mm to (412.2, 33.3), turned to 225 degrees
- moved C2 4.06 mm to (408.1, 33.4), turned to 90 degrees
- renumbered D_K0 to D_A6, D_K1 to D_A7, D_K2 to D_A8, D_K3 to D_A9, D_L0 to D_B6, D_L1 to D_B7, D_L2 to D_B8, D_L3 to D_B9, D_M0 to D_C6, D_M1 to D_C7, D_M2 to D_C8, D_M3 to D_C9, D_G5 to D_D5, D_N0 to D_D6, D_N1 to D_D7, D_N3 to D_D8, D_O0 to D_E6, D_O1 to D_E7, D_O2 to D_E8, D_O3 to D_E9, D_P0 to D_F6, D_P1 to D_F7, D_P2 to D_F8, D_P3 to D_F9, D_Q0 to D_G6, D_Q1 to D_G7, D_Q2 to D_G8, D_Q3 to D_G9, D_R0 to D_H6, D_R1 to D_H7, D_R2 to D_H8, D_R3 to D_H9, D_K5 to D_I5, D_N4 to D_I6, D_M4 to D_I7, D_L4 to D_I8, D_K4 to D_I9, D_R4 to D_J6, D_Q4 to D_J7, D_P4 to D_J8, D_O4 to D_J9, MX_K0 to MX_A6, MX_K1 to MX_A7, MX_K2 to MX_A8, MX_K3 to MX_A9, MX_L0 to MX_B6, MX_L1 to MX_B7, MX_L2 to MX_B8, MX_L3 to MX_B9, MX_M0 to MX_C6, MX_M1 to MX_C7, MX_M2 to MX_C8, MX_M3 to MX_C9, MX_G5 to MX_D5, MX_N0 to MX_D6, MX_N1 to MX_D7, MX_N3 to MX_D8, MX_M5 to MX_E5, MX_O0 to MX_E6, MX_O1 to MX_E7, MX_O2 to MX_E8, MX_O3 to MX_E9, MX_P0 to MX_F6, MX_P1 to MX_F7, MX_P2 to MX_F8, MX_P3 to MX_F9, MX_Q0 to MX_G6, MX_Q1 to MX_G7, MX_Q2 to MX_G8, MX_Q3 to MX_G9, MX_R0 to MX_H6, MX_R1 to MX_H7, MX_R2 to MX_H8, MX_R3 to MX_H9, MX_K5 to MX_I5, MX_N4 to MX_I6, MX_M4 to MX_I7, MX_L4 to MX_I8, MX_K4 to MX_I9, MX_R4 to MX_J6, MX_Q4 to MX_J7, MX_P4 to MX_J8, MX_O4 to MX_J9, MX_S0 to MX_K0, MX_S1 to MX_K1, MX_S3 to MX_K2, MX_S4 to MX_K3, MX_S5 to MX_K4, MX_R5 to MX_K5, MX_Q5 to MX_K6, MX_P5 to MX_K7, MX_N5 to MX_K8, MX_L5 to MX_K9
Connections:
- D_A6 pad 1: ROW0 -> ROW6
- D_A7 pad 1: ROW1 -> ROW7
- D_A8 pad 1: ROW2 -> ROW8
- D_A9 pad 1: ROW3 -> ROW9
- D_B6 pad 1: ROW0 -> ROW6
- D_B7 pad 1: ROW1 -> ROW7
- D_B8 pad 1: ROW2 -> ROW8
- D_B9 pad 1: ROW3 -> ROW9
- D_C6 pad 1: ROW0 -> ROW6
- D_C7 pad 1: ROW1 -> ROW7
- D_C8 pad 1: ROW2 -> ROW8
- D_C9 pad 1: ROW3 -> ROW9
- D_D6 pad 1: ROW0 -> ROW6
- D_D7 pad 1: ROW1 -> ROW7
- D_D8 pad 1: ROW3 -> ROW8
- D_E6 pad 1: ROW0 -> ROW6
- D_E7 pad 1: ROW1 -> ROW7
- D_E8 pad 1: ROW2 -> ROW8
- D_E9 pad 1: ROW3 -> ROW9
- D_F6 pad 1: ROW0 -> ROW6
- D_F7 pad 1: ROW1 -> ROW7
- D_F8 pad 1: ROW2 -> ROW8
- D_F9 pad 1: ROW3 -> ROW9
- D_G6 pad 1: ROW0 -> ROW6
- D_G7 pad 1: ROW1 -> ROW7
- D_G8 pad 1: ROW2 -> ROW8
- D_G9 pad 1: ROW3 -> ROW9
- D_H6 pad 1: ROW0 -> ROW6
- D_H7 pad 1: ROW1 -> ROW7
- D_H8 pad 1: ROW2 -> ROW8
- D_H9 pad 1: ROW3 -> ROW9
- D_I6 pad 1: ROW4 -> ROW6
- D_I7 pad 1: ROW4 -> ROW7
- D_I8 pad 1: ROW4 -> ROW8
- D_I9 pad 1: ROW4 -> ROW9
- D_J6 pad 1: ROW4 -> ROW6
- D_J7 pad 1: ROW4 -> ROW7
- D_J8 pad 1: ROW4 -> ROW8
- D_J9 pad 1: ROW4 -> ROW9
- D_L5 pad 1: ROW5 -> ROW9
- D_N5 pad 1: ROW5 -> ROW8
- D_P5 pad 1: ROW5 -> ROW7
- D_Q5 pad 1: ROW5 -> Net-(D_Q5-Pad1)
- D_S3 pad 1: ROW3 -> ROW2
- D_S4 pad 1: ROW4 -> ROW3
- D_S5 pad 1: ROW5 -> ROW4
- MX_A6 pad 1: COL_K -> COL_A
- MX_A7 pad 1: COL_K -> COL_A
- MX_A8 pad 1: COL_K -> COL_A
- MX_A9 pad 1: COL_K -> COL_A
- MX_B6 pad 1: COL_L -> COL_B
- MX_B7 pad 1: COL_L -> COL_B
- MX_B8 pad 1: COL_L -> COL_B
- MX_B9 pad 1: COL_L -> COL_B
- MX_C6 pad 1: COL_M -> COL_C
- MX_C7 pad 1: COL_M -> COL_C
- MX_C8 pad 1: COL_M -> COL_C
- MX_C9 pad 1: COL_M -> COL_C
- MX_D5 pad 1: COL_G -> COL_D
- MX_D6 pad 1: COL_N -> COL_D
- MX_D7 pad 1: COL_N -> COL_D
- MX_D8 pad 1: COL_N -> COL_D
- MX_E5 pad 1: COL_M -> COL_E
- MX_E6 pad 1: COL_O -> COL_E
- MX_E7 pad 1: COL_O -> COL_E
- MX_E8 pad 1: COL_O -> COL_E
- MX_E9 pad 1: COL_O -> COL_E
- MX_F6 pad 1: COL_P -> COL_F
- MX_F7 pad 1: COL_P -> COL_F
- MX_F8 pad 1: COL_P -> COL_F
- MX_F9 pad 1: COL_P -> COL_F
- MX_G6 pad 1: COL_Q -> COL_G
- MX_G7 pad 1: COL_Q -> COL_G
- MX_G8 pad 1: COL_Q -> COL_G
- MX_G9 pad 1: COL_Q -> COL_G
- MX_H6 pad 1: COL_R -> COL_H
- MX_H7 pad 1: COL_R -> COL_H
- MX_H8 pad 1: COL_R -> COL_H
- MX_H9 pad 1: COL_R -> COL_H
- MX_I5 pad 1: COL_K -> COL_I
- MX_I6 pad 1: COL_N -> COL_I
- MX_I7 pad 1: COL_M -> COL_I
- MX_I8 pad 1: COL_L -> COL_I
- MX_I9 pad 1: COL_K -> COL_I
- MX_J6 pad 1: COL_R -> COL_J
- MX_J7 pad 1: COL_Q -> COL_J
- MX_J8 pad 1: COL_P -> COL_J
- MX_J9 pad 1: COL_O -> COL_J
- MX_K0 pad 1: COL_S -> COL_K
- MX_K1 pad 1: COL_S -> COL_K
- MX_K2 pad 1: COL_S -> COL_K
- MX_K3 pad 1: COL_S -> COL_K
- MX_K4 pad 1: COL_S -> COL_K
- MX_K5 pad 1: COL_R -> COL_K
- MX_K6 pad 1: COL_Q -> COL_K
- MX_K7 pad 1: COL_P -> COL_K
- MX_K8 pad 1: COL_N -> COL_K
- MX_K9 pad 1: COL_L -> COL_K
- U1 pad 1: Net-(U1-Pad1) -> COL_F
- U1 pad 10: COL_R -> COL_B
- U1 pad 11: COL_Q -> COL_A
- U1 pad 12: COL_R -> Net-(U1-Pad12)
- U1 pad 18: ROW4 -> ROW0
- U1 pad 19: ROW3 -> COL_K
- U1 pad 20: ROW1 -> ROW2
- U1 pad 21: COL_P -> ROW4
- U1 pad 22: COL_M -> ROW5
- U1 pad 25: COL_N -> ROW3
- U1 pad 26: COL_O -> ROW1
- U1 pad 27: COL_K -> ROW6
- U1 pad 28: COL_L -> COL_J
- U1 pad 29: COL_J -> COL_H
- U1 pad 30: COL_G -> ROW8
- U1 pad 31: COL_C -> ROW7
- U1 pad 32: COL_B -> COL_I
- U1 pad 36: COL_A -> COL_E
- U1 pad 37: COL_I -> COL_G
- U1 pad 38: COL_H -> ROW9
- U1 pad 39: COL_F -> Net-(U1-Pad39)
- U1 pad 40: COL_E -> Net-(U1-Pad40)
- U1 pad 41: COL_D -> Net-(U1-Pad41)
- U1 pad 8: COL_S -> COL_D
- U1 pad 9: ROW5 -> COL_C
- U2 pad 6: Net-(U2-Pad6) -> (no net)
Routing:
- net ROW6: track 0.00 -> 404.9 mm, vias 0 -> 4
- net ROW7: track 0.00 -> 400.5 mm, vias 0 -> 9
- net ROW8: track 0.00 -> 395.2 mm, vias 0 -> 15
- net COL_L: track 364.1 -> 0.00 mm, vias 6 -> 0
- net COL_M: track 357.7 -> 0.00 mm, vias 1 -> 0
- net COL_N: track 321.9 -> 0.00 mm, vias 1 -> 0
- net ROW9: track 0.00 -> 320.3 mm, vias 0 -> 8
- net COL_O: track 300.7 -> 0.00 mm, vias 3 -> 0
- net COL_P: track 299.7 -> 0.00 mm, vias 8 -> 0
- net COL_R: track 295.0 -> 0.00 mm, vias 8 -> 0
- net COL_Q: track 194.1 -> 0.00 mm, vias 5 -> 0
- net COL_S: track 177.4 -> 0.00 mm, vias 3 -> 0
- net ROW2: track 365.4 -> 514.9 mm, vias 0 -> 10
- net COL_E: track 418.7 -> 553.1 mm, vias 2 -> 7
- net COL_D: track 454.3 -> 562.5 mm, vias 4 -> 7
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