File: keyboard_layout_jopr.kicad_pcb (KiCad board)
At the start: 2 copper layers, 428.6 x 123 mm, 229 parts, among them SW1 SW_Push, U1 ATmega32U4-AU, U2 SOT65P210X110, Y1 16MHz

Commit message: added LEDs for Lock keys
Parts:
- MX_E6, MX_F6, MX_G6: value MX-NoLED -> MX-LED-MX_Alps_Hybrid; footprint MX_Only:MXOnly-1U-NoLED -> MX_Only:MXOnly-1U-FLIPPED
Connections:
- U1 pad 39: Net-(U1-Pad39) -> LED_LEFT
- U1 pad 40: Net-(U1-Pad40) -> LED_MIDDLE
- U1 pad 41: Net-(U1-Pad41) -> LED_RIGHT
Routing:
- net LED_LEFT: track 0.00 -> 146.2 mm, vias 0 -> 7
- net LED_MIDDLE: track 0.00 -> 119.0 mm, vias 0 -> 3
- net LED_RIGHT: track 0.00 -> 97.3 mm, vias 0 -> 5
- net GND: track 418.9 -> 435.8 mm, vias 9 -> 12
- net ROW6: track 404.9 -> 409.6 mm

Commit message: removed NumLock
Parts:
- MX_E6: value MX-LED-MX_Alps_Hybrid -> MX-NoLED; footprint MX_Only:MXOnly-1U-FLIPPED -> MX_Only:MXOnly-1U-NoLED
Connections:
- U1 pad 39: LED_LEFT -> Net-(U1-Pad39)
Routing:
- net LED_LEFT: track 146.2 -> 0.00 mm, vias 7 -> 0
- net GND: track 435.8 -> 430.2 mm, vias 12 -> 11
