File: keyboard_layout_jopr.sch (KiCad schematic (older format))
At the start: 228 parts, among them SW1 SW_Push, U1 ATmega32U4-AU, Y1 16MHz

Commit message: Inter-key tracks and USB Data tracks only
Parts:
- renumbered D_O5 to D_P5, MX_O5 to MX_P5
Other:
- moved on the sheet: D_P5
Changed lines of the file:
@@
 EESchema Schematic File Version 4
+LIBS:keyboard_layout_jopr-cache
 EELAYER 29 0
 EELAYER END
@@
 $EndComp
 Wire Wire Line
-	9650 6150 9700 6150
+	10050 6150 10100 6150
 $Comp
-L Device:D_Small D_O5
+L Device:D_Small D_P5
 U 1 1 5EF0BE75
-P 9650 6250
-F 0 "D_O5" H 9650 6350 50  0000 R CNN
-F 1 "SOD-123" H 9700 6350 50  0000 L CNN
-F 2 "Diode_SMD:D_SOD-123" V 9650 6250 50  0001 C CNN
-F 3 "~" V 9650 6250 50  0001 C CNN
-	1    9650 6250
+P 10050 6250
+F 0 "D_P5" H 10050 6350 50  0000 R CNN
+F 1 "SOD-123" H 10100 6350 50  0000 L CNN
+F 2 "Diode_SMD:D_SOD-123" V 10050 6250 50  0001 C CNN
+F 3 "~" V 10050 6250 50  0001 C CNN
+	1    10050 6250
 	0    -1   -1   0
 $EndComp
 $Comp
-L MX_Alps_Hybrid:MX-NoLED MX_O5
+L MX_Alps_Hybrid:MX-NoLED MX_P5
 U 1 1 5EF0BE7B
-P 9750 6000
-F 0 "MX_O5" H 9783 6223 60  0000 C CNN
-F 1 "MX-NoLED" H 9783 6149 20  0000 C CNN
-F 2 "MX_Alps_Hybrid:MX-1U-NoLED" H 9125 5975 60  0001 C CNN
-F 3 "" H 9125 5975 60  0001 C CNN
-	1    9750 6000
+P 10150 6000
+F 0 "MX_P5" H 10183 6223 60  0000 C CNN
+F 1 "MX-NoLED" H 10183 6149 20  0000 C CNN
+F 2 "MX_Alps_Hybrid:MX-1U-NoLED" H 9525 5975 60  0001 C CNN
+F 3 "" H 9525 5975 60  0001 C CNN
+	1    10150 6000
 	1    0    0    -1
 $EndComp
 Wire Wire Line
 	9250 6150 9300 6150
-Wire Wire Line
-	9650 6350 9250 6350
 Connection ~ 9250 6350
 $Comp
@@
 $EndComp
 Wire Wire Line
-	9900 5300 9900 5950
-Connection ~ 9900 5300
+	10300 5300 10300 5950
 $Comp
 L MX_Alps_Hybrid:MX-NoLED MX_O4
@@
 $EndComp
 Connection ~ 10700 5300
-Connection ~ 9650 6350
-Wire Wire Line
-	9650 6350 10450 6350
 Wire Wire Line
 	10700 5300 10700 5950
@@
 Text GLabel 3150 2700 2    50   Input ~ 0
 COL_J
+Connection ~ 10050 6350
+Wire Wire Line
+	10050 6350 10450 6350
+Connection ~ 10300 5300
+Wire Wire Line
+	9250 6350 10050 6350
 $EndSCHEMATC

Commit message: maybe better tracks
Parts:
- MX_A0, MX_A1, MX_A2, MX_A3, MX_A4, MX_A5, MX_B0, MX_B1, MX_B2, MX_B3, MX_B4, MX_B5, MX_C0, MX_C1, MX_C2, MX_C3, MX_C4, MX_C5, MX_D0, MX_D1, MX_D2, MX_D3, MX_D4, MX_E0, MX_E1, MX_E2, MX_E3, MX_E4, MX_F0, MX_F1, MX_F2, MX_F3, MX_F4, MX_G0, MX_G1, MX_G2, MX_G3, MX_G4, MX_G5, MX_H0, MX_H1, MX_H2, MX_H3, MX_H4, MX_I0, MX_I1, MX_I2, MX_I3, MX_I4, MX_J0, MX_J1, MX_J2, MX_J3, MX_J4, MX_J5, MX_K0, MX_K1, MX_K2, MX_K3, MX_K4, MX_K5, MX_L0, MX_L1, MX_L2, MX_L3, MX_L4, MX_L5, MX_M0, MX_M1, MX_M2, MX_M3, MX_M4, MX_M5, MX_N0, MX_N1, MX_N3, MX_N4, MX_N5, MX_O1, MX_O2, MX_O3, MX_O4, MX_P1, MX_P2, MX_P3, MX_P4, MX_P5, MX_Q1, MX_Q2, MX_Q3, MX_Q4, MX_Q5, MX_R0, MX_R1, MX_R2, MX_R3, MX_R4, MX_R5, MX_S0, MX_S1, MX_S3, MX_S4, MX_S5: symbol MX_Alps_Hybrid:MX-NoLED -> keyboard_layout_jopr-rescue:MX-NoLED-MX_Alps_Hybrid
- MX_O0, MX_P0, MX_Q0: symbol MX_Alps_Hybrid:MX-LED -> keyboard_layout_jopr-rescue:MX-LED-MX_Alps_Hybrid
- USB1: symbol random-keyboard-parts:Molex-0548190589 -> keyboard_layout_jopr-rescue:Molex-0548190589-random-keyboard-parts
